Commit message: Initial commit of dual camera docking.

File: models/multigo/multigo.urdf (robot description, URDF)
Before this commit: robot multigo, 12 links, 11 joints
Links:
- removed link camera_front_frame
- removed link camera_left_frame
- removed link camera_right_frame
- added link camera_front_left_frame, mass 0.5; collision box size=0.1 0.1 0.1; visual box size=0.1 0.1 0.1
- added link camera_front_right_frame, mass 0.5; collision box size=0.1 0.1 0.1; visual box size=0.1 0.1 0.1
Joints:
- removed joint camera_front_joint
- removed joint camera_left_joint
- removed joint camera_right_joint
- added joint camera_front_left_joint: type fixed, parent camera_link, child camera_front_left_frame, origin xyz=-0.082 0.178 0.0 rpy=0 0 0
- added joint camera_front_right_joint: type fixed, parent camera_link, child camera_front_right_frame, origin xyz=-0.082 -0.178 0.0 rpy=0 0 0
